Commit message: Atualizou bioloid_example com cabeça

File: bioloid_example/urdf/bioloid_torso_std_part.xacro (robot description, xacro)
@@ -17,8 +17,10 @@
         </visual>
         <!-- Sensor 100 -->
+        <!--
         <visual>
             <xacro:default_geometry cad_file="AX-S1"/>
             <origin xyz="0 0 0.025" rpy="${-pi/2} 0 ${pi}"/>
         </visual>
+        -->
         <!-- Motor 1 -->
         <visual>

File: bioloid_example/urdf/bioloid_without_legs.xacro (robot description, xacro)
@@ -64,5 +64,5 @@
     <!-- World -->
     <!-- Used for fixing robot to Gazebo 'base_link' -->
-      <link name="world"/>
+    <link name="world"/>
       <joint name="fixed" type="fixed">
         <parent link="world"/>
@@ -78,4 +78,76 @@
     <link name="base_link">
     </link>
+    <!-- Neck Joint-->
+  <joint
+    name="head_yaw_joint"
+    type="revolute">
+    <origin
+      xyz="0 0 0.015"
+      rpy="0 0 0" />
+    <parent
+      link="base_link" />
+    <child
+      link="neck_link" />
+    <limit lower="${-pi}" upper="${pi}" effort="10" velocity="1.0"/>
+    <axis
+      xyz="0 0 1" />
+    <limit
+      effort="0"
+      velocity="0" />
+  </joint>
+  <!-- Neck Link-->
+    <link
+    name="neck_link">
+    <visual>
+      <origin
+        xyz="0 0 0"
+        rpy="0 0 0" />
+      <geometry>
+        <mesh
+          filename="package://bioloid_example/mesh/neck_link.STL" />
+      </geometry>
+      <material
+        name="">
+        <color
+          rgba="0.1 0.1 0.1 1" />
+      </material>
+    </visual>
+  </link>
+    <!-- Head Link-->
+  <link
+    name="head_link">
+    <visual>
+      <origin
+        xyz="0 0 0"
+        rpy="0 0 0" />
+      <geometry>
+        <mesh
+          filename="package://bioloid_example/mesh/head_link.STL" />
+      </geometry>
+      <material
+        name="">
+        <color
+          rgba="0.5 0.5 0.5 1" />
+      </material>
+    </visual>
+  </link>
+  <!-- Head Joint-->
+  <joint
+    name="head_pitch_joint"
+    type="revolute">
+    <origin
+      xyz="0.008 0 0.053"
+      rpy="0 0 0" />
+    <parent
+      link="neck_link" />
+    <child
+      link="head_link" />
+      <limit lower="-1.3" upper="1.4" effort="10" velocity="1.0"/>
+    <axis
+      xyz="0 1 0" />
+    <limit
+      effort="0"
+      velocity="0" />
+  </joint>
     <!-- Torso to right shoulder -->
     <xacro:shoulder_swing_joint prefix="right" reflect="1"/>
