Commit message: Separou código de teste do dxl_robot_hw_test e do bioloid_example

File: bioloid_example/urdf/bioloid_without_legs.xacro (robot description, xacro)
@@ -65,9 +65,28 @@
     <!-- Used for fixing robot to Gazebo 'base_link' -->
     <link name="world"/>
-      <joint name="fixed" type="fixed">
+    <joint name="world_to_odom" type="fixed">
         <parent link="world"/>
-        <child link="base_link"/>
+        <child link="odom"/>
         <origin xyz="0 0 0.3" rpy="0 0 0"/>
       </joint>
+    <link name="odom"/>
+      <joint name="odom_to_imu" type="fixed">
+        <parent link="odom"/>
+        <child link="imu"/>
+        <origin xyz="0 0 0" rpy="0 0 0"/>
+      </joint>
+    <link name="imu"/>
+      <joint name="imu_to_base_link" type="fixed">
+        <parent link="imu"/>
+        <child link="base_link"/>
+        <origin xyz="0 0 0" rpy="0 0 0"/>
+      </joint>
+<!--
+    <joint name="imu_to_base" type="fixed">
+        <parent link="imu"/>
+        <child link="base_link"/>
+        <origin xyz="0 0 0" rpy="0 0 0"/>
+      </joint>
+-->
     <!-- Base -->
     <joint name="base_to_torso_joint" type="fixed">

Commit message: Ajustes de organização de código

File: bioloid_example/urdf/bioloid_without_legs.xacro (robot description, xacro)
@@ -80,5 +80,5 @@
         <parent link="imu"/>
         <child link="base_link"/>
-        <origin xyz="0 0 0" rpy="0 0 0"/>
+        <origin xyz="0 0 0" rpy="0 0 ${pi/2}"/>
       </joint>
 <!--
